Commit message: added upper body (RM arms)

File: urdf/bit_humanoid.urdf (robot description, URDF)
Before this commit: robot bit_humanoid, 20 links, 19 joints
Links:
- added link LArm2, mass 0.43285; collision mesh filename=package://bit_humanoid/meshes/LArm2.STL; visual mesh filename=package://bit_humanoid/meshes/LArm2.STL
- added link LArm3, mass 0.43132; collision mesh filename=package://bit_humanoid/meshes/LArm3.STL; visual mesh filename=package://bit_humanoid/meshes/LArm3.STL
- added link LArm4, mass 0.28963; collision mesh filename=package://bit_humanoid/meshes/LArm4.STL; visual mesh filename=package://bit_humanoid/meshes/LArm4.STL
- added link LArm5, mass 0.23941; collision mesh filename=package://bit_humanoid/meshes/LArm5.STL; visual mesh filename=package://bit_humanoid/meshes/LArm5.STL
- added link LArm6, mass 0.21879; collision mesh filename=package://bit_humanoid/meshes/LArm6.STL; visual mesh filename=package://bit_humanoid/meshes/LArm6.STL
- added link LArm7, mass 0.14433; collision mesh filename=package://bit_humanoid/meshes/LArm7.STL; visual mesh filename=package://bit_humanoid/meshes/LArm7.STL
- added link RArm2, mass 0.43285; collision mesh filename=package://bit_humanoid/meshes/RArm2.STL; visual mesh filename=package://bit_humanoid/meshes/RArm2.STL
- added link RArm3, mass 0.43132; collision mesh filename=package://bit_humanoid/meshes/RArm3.STL; visual mesh filename=package://bit_humanoid/meshes/RArm3.STL
- added link RArm4, mass 0.28963; collision mesh filename=package://bit_humanoid/meshes/RArm4.STL; visual mesh filename=package://bit_humanoid/meshes/RArm4.STL
- added link RArm5, mass 0.23941; collision mesh filename=package://bit_humanoid/meshes/RArm5.STL; visual mesh filename=package://bit_humanoid/meshes/RArm5.STL
- added link RArm6, mass 0.21879; collision mesh filename=package://bit_humanoid/meshes/RArm6.STL; visual mesh filename=package://bit_humanoid/meshes/RArm6.STL
- added link RArm7, mass 0.14433; collision mesh filename=package://bit_humanoid/meshes/RArm7.STL; visual mesh filename=package://bit_humanoid/meshes/RArm7.STL
Joints:
- added joint LArm2: type revolute, parent LArm1, child LArm2, origin xyz=0 0 0 rpy=1.5708 0 0, axis 0 1 0, limit lower=-2.269 upper=2.269 effort=60 velocity=1
- added joint LArm3: type revolute, parent LArm2, child LArm3, origin xyz=0 0 0.256 rpy=-1.5708 0 0, axis 0 -1 0, limit lower=-3.107 upper=3.107 effort=10 velocity=1
- added joint LArm4: type revolute, parent LArm3, child LArm4, origin xyz=0 0 0 rpy=1.5708 0 0, axis 0 1 0, limit lower=-2.356 upper=2.356 effort=30 velocity=1
- added joint LArm5: type revolute, parent LArm4, child LArm5, origin xyz=0 0 0.21 rpy=-1.5708 0 0, axis 0 -1 0, limit lower=-3.107 upper=3.107 effort=10 velocity=1
- added joint LArm6: type revolute, parent LArm5, child LArm6, origin xyz=0 0 0 rpy=1.5708 0 0, axis 0 1 0, limit lower=-2.234 upper=2.234 effort=10 velocity=1
- added joint LArm7: type revolute, parent LArm6, child LArm7, origin xyz=0 0 0.1725 rpy=0 0 0, axis 0 0 1, limit lower=-6.283 upper=6.283 effort=10 velocity=1
- added joint RArm2: type revolute, parent RArm1, child RArm2, origin xyz=0 0 0 rpy=1.5708 0 0, axis 0 1 0, limit lower=-2.269 upper=2.269 effort=60 velocity=1
- added joint RArm3: type revolute, parent RArm2, child RArm3, origin xyz=0 0 0.256 rpy=-1.5708 0 0, axis 0 -1 0, limit lower=-3.107 upper=3.107 effort=10 velocity=1
- added joint RArm4: type revolute, parent RArm3, child RArm4, origin xyz=0 0 0 rpy=1.5708 0 0, axis 0 1 0, limit lower=-2.356 upper=2.356 effort=30 velocity=1
- added joint RArm5: type revolute, parent RArm4, child RArm5, origin xyz=0 0 0.21 rpy=-1.5708 0 0, axis 0 -1 0, limit lower=-3.107 upper=3.107 effort=10 velocity=1
- added joint RArm6: type revolute, parent RArm5, child RArm6, origin xyz=0 0 0 rpy=1.5708 0 0, axis 0 1 0, limit lower=-2.234 upper=2.234 effort=10 velocity=1
- added joint RArm7: type revolute, parent RArm6, child RArm7, origin xyz=0 0 0.1725 rpy=0 0 0, axis 0 0 1, limit lower=-6.283 upper=6.283 effort=10 velocity=1
